File: Datsun Gauges Fan Relay Driver.kicad_sch (KiCad schematic)
At the start: 8 parts, among them K1 RAYEX-L90AS, M1 Fan, Q1 IRL2203N or MTP3055VL, SW1 External Fan Sw

Commit message: Updated kicad diagrams
Updated kicad diagrams
Other:
- note added: "10k pulldown may not needed when using builtin LED pin since it has a resistor and LED to ground on SOME arduinos"
- note removed: "10k pulldown not needed when using builtin LED pin since it has a resistor and LED to ground"
Changed lines of the file:
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@@
     (stroke (width 0) (type default))
   )
-  (wire (pts (xy 176.53 81.28) (xy 193.04 81.28))
+  (wire (pts (xy 175.26 81.28) (xy 193.04 81.28))
     (stroke (width 0) (type default))
   )
@@
     (stroke (width 0) (type default))
   )
-  (text "10k pulldown not needed\nwhen using builtin LED pin\nsince it has a resistor\nand LED to ground"
+  (text "10k pulldown may not needed\nwhen using builtin LED pin\nsince it has a resistor\nand LED to ground on SOME arduinos"
     (at 91.44 107.95 0)
     (effects (font (size 1.27 1.27)) (justify left bottom))
