File: Datsun Gauges Fuel Temp Inputs.kicad_sch (KiCad schematic)
At the start: 29 parts, among them J1 Conn_01x03_Pin, J2 Conn_01x03_Socket, U1 LM358, U2 DS18B20

Commit message: Updated kicad diagrams
Updated kicad diagrams
Parts:
- R9: value 3k3 -> 2k2
Changed lines of the file:
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@@
       (effects (font (size 1.27 1.27)) (justify left))
     )
-    (property "Value" "3k3" (at 113.03 149.86 0)
+    (property "Value" "2k2" (at 113.03 149.86 0)
       (effects (font (size 1.27 1.27)) (justify left))
     )

Commit message: Cleanup
Other:
- moved on the sheet: C1, C2, C3, D1, D2, D3, D4, D5, R11, R9
