File: Datsun Gauges Power Supply.kicad_sch (KiCad schematic)
At the start: 22 parts, among them U1 LM2940CT-5 5v 1A, U2 Arduino adjustable SwPSU

Commit message: Updated kicad diagrams
Updated kicad diagrams
Parts:
- removed C4, C5: 2.2u 630VDC Polyester, symbol Device:C
- added C11: 2.2u 630VDC Polyester, symbol Device:C
- added C12, C13: 100n 50v Ceramic, symbol Device:C
- added C4, C5: 4.7uF 35v TT, symbol Device:C_Polarized
Connections:
- net Filtered IGN+: now also C4.1
Other:
- moved on the sheet: C1, C10

Commit message: Cleanup
Other:
- moved on the sheet: C1, C11, C2, C3, C4, C5, C7, D1, D2, D5, D6
